File: ECAD/DnD20/DnD20.sch (KiCad schematic (older format))
At the start: 38 parts, among them IC1g$1 CP2104, J1 Conn_01x03_Female, J2 Conn_01x04_Female, Q1 2N2219, Q2 2N2219, SW1 switch, SW2 switch, U1 ESP12, U2 AP2112-3.3, U3 MCP73831/2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

Commit message: Refactored firmware before removing accelerometer
Parts:
- IC1g$1: symbol DnD20:CP2104 -> DnD20-rescue:CP2104-DnD20
- SW1, SW2: symbol DnD20:switch -> DnD20-rescue:switch-DnD20
- U1: symbol DnD20:ESP12 -> DnD20-rescue:ESP12-DnD20
- U2: symbol DnD20:AP2112-3.3 -> DnD20-rescue:AP2112-3.3-DnD20
- U3: symbol DnD20:MCP73831_2 -> DnD20-rescue:MCP73831_2-DnD20
- X1: symbol DnD20:JSTPH -> DnD20-rescue:JSTPH-DnD20
Changed lines of the file:
@@
 $EndDescr
 $Comp
-L DnD20:AP2112-3.3 U2
+L DnD20-rescue:AP2112-3.3-DnD20 U2
 U 1 1 5ABE7420
 P 2150 2000
@@
 $EndComp
 $Comp
-L DnD20:switch SW2
+L DnD20-rescue:switch-DnD20 SW2
 U 1 1 5ABE9F7C
 P 4150 1950
@@
 $EndComp
 $Comp
-L DnD20:CP2104 IC1g$1
+L DnD20-rescue:CP2104-DnD20 IC1g$1
 U 1 1 5ABEAC9C
 P 7350 2000
@@
 	4800 3550 11250 3550
 $Comp
-L DnD20:ESP12 U1
+L DnD20-rescue:ESP12-DnD20 U1
 U 1 1 5ABEC30E
 P 1650 4050
@@
 	2250 4150 2850 4150
 $Comp
-L DnD20:JSTPH X1
+L DnD20-rescue:JSTPH-DnD20 X1
 U 1 1 5ABEC8FB
 P 2700 1150
@@
 	5450 5750 500  5750
 $Comp
-L DnD20:MCP73831_2 U3
+L DnD20-rescue:MCP73831_2-DnD20 U3
 U 1 1 5ABF4440
 P 2150 6700
@@
 $EndComp
 $Comp
-L DnD20:switch SW1
+L DnD20-rescue:switch-DnD20 SW1
 U 1 1 5BC18FE1
 P 10000 2700
